Commit message: added urdf link

File: urdf/FFS055YA501U6.xacro (robot description, xacro)
@@ -1,26 +1,20 @@
 <?xml version="1.0"?>
-<robot xmlns:xacro="http://www.ros.org/wiki/xacro">
+<robot name="FFS055YA501U6" xmlns:xacro="http://www.ros.org/wiki/xacro">
     <joint name="base_joint" type="fixed">
         <origin xyz="0 0 0" rpy="0 0 0" />
         <parent link="base_link" />
-        <child link="sensor" />
+        <child link="sensor_link" />
     </joint>
     <link name="base_link" />
-    <link name="ffs055ya501u6_link">
-        <inertial>
-        </inertial>
+    <link name="sensor_link">
         <visual>
-            <origin xyz="0 0 0" rpy="0 0 0" />
+            <origin xyz="0 0 -0.01" rpy="1.57079 0 0" />
             <geometry>
                 <mesh filename="package://leptrino_force_torque/meshes/FFS055YA501U6.stl" />
             </geometry>
-            <material name="grey"/>
+            <material name="grey">
+                <color rgba="0.7 0.7 0.7 1.0" />
+            </material>
         </visual>
-        <collision>
-            <origin xyz="0 0 0" rpy="0 0 0" />
-            <geometry>
-                <mesh filename="package://leptrino_force_torque/meshes/FFS055YA501U6.stl" />
-            </geometry>
-        </collision>
     </link>
 </robot>

Commit message: setup rviz

File: urdf/FFS055YA501U6.xacro (robot description, xacro)
@@ -1,11 +1,11 @@
 <?xml version="1.0"?>
 <robot name="FFS055YA501U6" xmlns:xacro="http://www.ros.org/wiki/xacro">
-    <joint name="base_joint" type="fixed">
+    <joint name="leptrino_joint" type="fixed">
         <origin xyz="0 0 0" rpy="0 0 0" />
         <parent link="base_link" />
-        <child link="sensor_link" />
+        <child link="leptrino" />
     </joint>
     <link name="base_link" />
-    <link name="sensor_link">
+    <link name="leptrino">
         <visual>
             <origin xyz="0 0 -0.01" rpy="1.57079 0 0" />
