Commit message: fix bug

File: urdf/contact_device_v1.xacro (robot description, xacro)
@@ -4,13 +4,13 @@
         <origin xyz="0 0 0" rpy="0 0 0" />
         <parent link="base_link" />
-        <child link="sensor_link" />
+        <child link="leptrino" />
     </joint>
     <joint name="contact_joint" type="fixed">
         <origin xyz="0 0 0" rpy="0 0 0" />
-        <parent link="sensor_link" />
+        <parent link="leptrino" />
         <child link="contact_link" />
     </joint>
     <link name="base_link" />
-    <link name="sensor_link">
+    <link name="leptrino">
         <visual>
             <origin xyz="0 0 -0.01" rpy="1.57079 0 0" />
